Commit message: update holder angle

File: midem_description/urdf/midem_with_solder_lead.xacro (robot description, xacro)
@@ -24,8 +24,8 @@
     <origin xyz="0 0 0" rpy="0 0 0"/>
   </joint>
-	<link name="clip_base">
+  <link name="clip_base">
     <visual>
       <geometry>
-  			<mesh filename="${mesh_path2}/holder/meshes/clip_base.dae" scale="${mesh_scale2}"/>
+  		<mesh filename="${mesh_path2}/holder/meshes/clip_base.dae" scale="${mesh_scale2}"/>
       </geometry>
       <origin rpy="3.141592 0 1.570796" xyz="-0.01 0 0.015"/>
@@ -41,10 +41,10 @@
     <parent link="force_sensor_base"/>
     <child link="clip_base"/>
-    <origin xyz="0 0 0.068" rpy="0 -0.2 0"/>
+    <origin xyz="0 0 0.068" rpy="0 -0.3 0"/>
   </joint>
   <link name="clip_cover">
     <visual>
       <geometry>
-  			<mesh filename="${mesh_path2}/holder/meshes/clip_cover.dae" scale="${mesh_scale2}"/>
+  		<mesh filename="${mesh_path2}/holder/meshes/clip_cover.dae" scale="${mesh_scale2}"/>
       </geometry>
       <origin rpy="0 0 1.570796" xyz="0.01 0 0"/>
@@ -65,5 +65,5 @@
     <visual>
       <geometry>
-  			<cylinder radius="0.01" length="0.095"/>
+  		<cylinder radius="0.01" length="0.095"/>
       </geometry>
       <material name="Cyan">
@@ -74,5 +74,5 @@
     <collision>
       <geometry>
-  			<cylinder radius="0.011" length="0.11"/>
+  		<cylinder radius="0.011" length="0.11"/>
       </geometry>
       <origin rpy="0 0 0" xyz="0 0 -0.0475"/>
